Commit message: Revisión de URDF files

File: abb_irb2400/urdf/irb2400.urdf (robot description, URDF)
Before this commit: robot abb_irb2400, 9 links, 8 joints
Links:
- link base_link: geometry collision mesh filename=/home/stmark/robot_arm_ws/src/abb_irb2400/meshes/irb2400/co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; visual mesh filename=/home/stmark/robot_arm_ws/src/abb_irb2400/meshes/irb2400/vi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
- link link_1: geometry collision mesh filename=/home/stmark/robot_arm_ws/src/abb_irb2400/meshes/irb2400/co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; visual mesh filename=/home/stmark/robot_arm_ws/src/abb_irb2400/meshes/irb2400/vi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
- link link_2: geometry collision mesh filename=/home/stmark/robot_arm_ws/src/abb_irb2400/meshes/irb2400/co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; visual mesh filename=/home/stmark/robot_arm_ws/src/abb_irb2400/meshes/irb2400/vi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
- link link_3: geometry collision mesh filename=/home/stmark/robot_arm_ws/src/abb_irb2400/meshes/irb2400/co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; visual mesh filename=/home/stmark/robot_arm_ws/src/abb_irb2400/meshes/irb2400/vi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
- link link_4: geometry collision mesh filename=/home/stmark/robot_arm_ws/src/abb_irb2400/meshes/irb2400/co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; visual mesh filename=/home/stmark/robot_arm_ws/src/abb_irb2400/meshes/irb2400/vi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
- link link_5: geometry collision mesh filename=/home/stmark/robot_arm_ws/src/abb_irb2400/meshes/irb2400/co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; visual mesh filename=/home/stmark/robot_arm_ws/src/abb_irb2400/meshes/irb2400/vi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
- link link_6: geometry collision mesh filename=/home/stmark/robot_arm_ws/src/abb_irb2400/meshes/irb2400/co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; visual mesh filename=/home/stmark/robot_arm_ws/src/abb_irb2400/meshes/irb2400/vi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

Commit message: Añadiendo archivos launch abb

File: abb_irb2400/urdf/irb2400.urdf (robot description, URDF)
Before this commit: robot abb_irb2400, 9 links, 8 joints
Links:
- link base_link: geometry collision mesh filename=package://abb_irb2400/meshes/irb2400/collision/base_link.stl; visual mesh filename=package://abb_irb2400/meshes/irb2400/visual/base_link.dae
- link link_1: geometry collision mesh filename=package://abb_irb2400/meshes/irb2400/collision/link_1.stl; visual mesh filename=package://abb_irb2400/meshes/irb2400/visual/link_1.dae
- link link_2: geometry collision mesh filename=package://abb_irb2400/meshes/irb2400/collision/link_2_whole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; visual mesh filename=package://abb_irb2400/meshes/irb2400/visual/link_2.dae
- link link_3: geometry collision mesh filename=package://abb_irb2400/meshes/irb2400/collision/link_3.stl; visual mesh filename=package://abb_irb2400/meshes/irb2400/visual/link_3.dae
- link link_4: geometry collision mesh filename=package://abb_irb2400/meshes/irb2400/collision/link_4.stl; visual mesh filename=package://abb_irb2400/meshes/irb2400/visual/link_4.dae
- link link_5: geometry collision mesh filename=package://abb_irb2400/meshes/irb2400/collision/link_5.stl; visual mesh filename=package://abb_irb2400/meshes/irb2400/visual/link_5.dae
- link link_6: geometry collision mesh filename=package://abb_irb2400/meshes/irb2400/collision/link_6.stl; visual mesh filename=package://abb_irb2400/meshes/irb2400/visual/link_6.dae

File: kuka_kr210_arm/urdf/kr210.urdf (robot description, URDF)
Before this commit: robot kuka_kr210_arm, 11 links, 10 joints
Links:
- link base_link: geometry collision mesh filename=package://kuka_kr210_arm/meshes/collision/base_link.stl; visual mesh filename=package://kuka_kr210_arm/meshes/visual/base_link.dae
- link gripper_link: geometry collision mesh filename=package://kuka_kr210_arm/meshes/visual/gripper_base.dae; visual mesh filename=package://kuka_kr210_arm/meshes/visual/gripper_base.dae
- link left_gripper_finger_link: geometry collision mesh filename=package://kuka_kr210_arm/meshes/collision/finger_left_colli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; visual mesh filename=package://kuka_kr210_arm/meshes/visual/finger_left.dae
- link link_1: geometry collision mesh filename=package://kuka_kr210_arm/meshes/collision/link_1.stl; visual mesh filename=package://kuka_kr210_arm/meshes/visual/link_1.dae
- link link_2: geometry collision mesh filename=package://kuka_kr210_arm/meshes/collision/link_2.stl; visual mesh filename=package://kuka_kr210_arm/meshes/visual/link_2.dae
- link link_3: geometry collision mesh filename=package://kuka_kr210_arm/meshes/collision/link_3.stl; visual mesh filename=package://kuka_kr210_arm/meshes/visual/link_3.dae
- link link_4: geometry collision mesh filename=package://kuka_kr210_arm/meshes/collision/link_4.stl; visual mesh filename=package://kuka_kr210_arm/meshes/visual/link_4.dae
- link link_5: geometry collision mesh filename=package://kuka_kr210_arm/meshes/collision/link_5.stl; visual mesh filename=package://kuka_kr210_arm/meshes/visual/link_5.dae
- link link_6: geometry collision mesh filename=package://kuka_kr210_arm/meshes/collision/link_6.stl; visual mesh filename=package://kuka_kr210_arm/meshes/visual/link_6.dae
- link right_gripper_finger_link: geometry collision mesh filename=package://kuka_kr210_arm/meshes/collision/finger_right_coll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; visual mesh filename=package://kuka_kr210_arm/meshes/visual/finger_right.dae

Commit message: Se añadieron las palancas al urdf

File: abb_irb2400/urdf/irb2400.urdf (robot description, URDF)
Before this commit: robot abb_irb2400, 9 links, 8 joints
Links:
- added link link_lever_a; collision mesh filename=package://abb_irb2400/meshes/irb2400/collision/link_lever_a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; visual mesh filename=package://abb_irb2400/meshes/irb2400/visual/link_lever_a.dae
- added link link_lever_b; collision mesh filename=package://abb_irb2400/meshes/irb2400/collision/link_lever_b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; visual mesh filename=package://abb_irb2400/meshes/irb2400/visual/link_lever_b.dae
Joints:
- added joint joint_lever_a: type continuous, parent link_2, child link_lever_a, origin xyz=0 0 0 rpy=0 0 0, axis 0 1 0, mimic joint=joint_3 multiplier=1.0
- added joint joint_lever_b: type continuous, parent link_3, child link_lever_b, origin xyz=-0.18 0 0 rpy=0 0 0, axis 0 1 0, mimic joint=joint_3 multiplier=-1.0

Commit message: Se arreglo la junta fuera de posición

File: abb_irb2400/urdf/irb2400.urdf (robot description, URDF)
Before this commit: robot abb_irb2400, 11 links, 10 joints
Joints:
- joint joint_4: origin xyz=0.258 0 0.135 rpy=0 0 0 -> xyz=0 0 0.135 rpy=0 0 0
- joint joint_5: origin xyz=0.497 0 0 rpy=0 0 0 -> xyz=0.755 0 0 rpy=0 0 0
